File: V1/usb tester.brd (EAGLE design)
At the start: 61 x 30.5 mm, 35 parts, among them T1 BC847, T2 BC847, T3 BC847, T4 BC847

Commit message: values
Parts:
- R1, R10, R11, R12, R13, R2, R3, R4: value (none) -> 1k2
- R5, R6, R7, R8, R9: value (none) -> 4k7
Changed lines of the file:
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@@
 </autorouter>
 <elements>
-<element name="R1" library="rcl" package="R0603" value="" x="24.13" y="26.67" smashed="yes" rot="R270">
+<element name="R1" library="rcl" package="R0603" value="1k2" x="24.13" y="26.67" smashed="yes" rot="R270">
 <attribute name="NAME" x="24.765" y="29.337" size="0.8128" layer="25" font="vector" ratio="12" rot="R180"/>
 <attribute name="VALUE" x="21.59" y="27.94" size="1.27" layer="27" rot="R270"/>
 </element>
-<element name="R2" library="rcl" package="R0603" value="" x="24.13" y="11.43" smashed="yes" rot="R270">
+<element name="R2" library="rcl" package="R0603" value="1k2" x="24.13" y="11.43" smashed="yes" rot="R270">
 <attribute name="NAME" x="24.765" y="14.097" size="0.8128" layer="25" font="vector" ratio="12" rot="R180"/>
 <attribute name="VALUE" x="21.59" y="12.7" size="1.27" layer="27" rot="R270"/>
 </element>
-<element name="R3" library="rcl" package="R0603" value="" x="24.13" y="16.51" smashed="yes" rot="R270">
+<element name="R3" library="rcl" package="R0603" value="1k2" x="24.13" y="16.51" smashed="yes" rot="R270">
 <attribute name="NAME" x="24.765" y="19.177" size="0.8128" layer="25" font="vector" ratio="12" rot="R180"/>
 <attribute name="VALUE" x="21.59" y="17.78" size="1.27" layer="27" rot="R270"/>
 </element>
-<element name="R4" library="rcl" package="R0603" value="" x="24.13" y="21.59" smashed="yes" rot="R270">
+<element name="R4" library="rcl" package="R0603" value="1k2" x="24.13" y="21.59" smashed="yes" rot="R270">
 <attribute name="NAME" x="24.765" y="24.257" size="0.8128" layer="25" font="vector" ratio="12" rot="R180"/>
 <attribute name="VALUE" x="21.59" y="22.86" size="1.27" layer="27" rot="R270"/>
@@
 <attribute name="NAME" x="38.735" y="24.257" size="0.8128" layer="25" font="vector" ratio="12" rot="R180"/>
 </element>
-<element name="R5" library="rcl" package="R0603" value="" x="29.21" y="26.67" smashed="yes" rot="R270">
+<element name="R5" library="rcl" package="R0603" value="4k7" x="29.21" y="26.67" smashed="yes" rot="R270">
 <attribute name="NAME" x="29.845" y="29.337" size="0.8128" layer="25" font="vector" ratio="12" rot="R180"/>
 <attribute name="VALUE" x="26.67" y="27.94" size="1.27" layer="27" rot="R270"/>
 </element>
-<element name="R6" library="rcl" package="R0603" value="" x="29.21" y="11.43" smashed="yes" rot="R270">
+<element name="R6" library="rcl" package="R0603" value="4k7" x="29.21" y="11.43" smashed="yes" rot="R270">
 <attribute name="NAME" x="29.845" y="14.097" size="0.8128" layer="25" font="vector" ratio="12" rot="R180"/>
 <attribute name="VALUE" x="26.67" y="12.7" size="1.27" layer="27" rot="R270"/>
 </element>
-<element name="R7" library="rcl" package="R0603" value="" x="29.21" y="16.51" smashed="yes" rot="R270">
+<element name="R7" library="rcl" package="R0603" value="4k7" x="29.21" y="16.51" smashed="yes" rot="R270">
 <attribute name="NAME" x="29.845" y="19.177" size="0.8128" layer="25" font="vector" ratio="12" rot="R180"/>
 <attribute name="VALUE" x="26.67" y="17.78" size="1.27" layer="27" rot="R270"/>
 </element>
-<element name="R8" library="rcl" package="R0603" value="" x="29.21" y="21.59" smashed="yes" rot="R270">
+<element name="R8" library="rcl" package="R0603" value="4k7" x="29.21" y="21.59" smashed="yes" rot="R270">
 <attribute name="NAME" x="29.845" y="24.257" size="0.8128" layer="25" font="vector" ratio="12" rot="R180"/>
 <attribute name="VALUE" x="26.67" y="22.86" size="1.27" layer="27" rot="R270"/>
@@
 <attribute name="NAME" x="47.625" y="22.606" size="0.8128" layer="25" font="vector" ratio="12"/>
 </element>
-<element name="R9" library="rcl" package="R0603" value="" x="49.53" y="13.335" smashed="yes">
+<element name="R9" library="rcl" package="R0603" value="4k7" x="49.53" y="13.335" smashed="yes">
 <attribute name="NAME" x="48.895" y="11.43" size="0.8128" layer="25" font="vector" ratio="12"/>
 <attribute name="VALUE" x="48.26" y="10.795" size="1.27" layer="27"/>
@@
 <attribute name="PROD_ID" value="CONN-09520" x="11.43" y="10.16" size="1.016" layer="28" font="vector" rot="MR90" display="off"/>
 </element>
-<element name="R10" library="rcl" package="R0603" value="" x="31.75" y="26.67" smashed="yes" rot="R90">
+<element name="R10" library="rcl" package="R0603" value="1k2" x="31.75" y="26.67" smashed="yes" rot="R90">
 <attribute name="NAME" x="32.766" y="29.337" size="0.8128" layer="25" font="vector" ratio="12" rot="R180"/>
 <attribute name="VALUE" x="34.29" y="25.4" size="1.27" layer="27" rot="R90"/>
@@
 <attribute name="VALUE" x="33.02" y="24.13" size="1.27" layer="27"/>
 </element>
-<element name="R11" library="rcl" package="R0603" value="" x="31.75" y="11.43" smashed="yes" rot="R90">
+<element name="R11" library="rcl" package="R0603" value="1k2" x="31.75" y="11.43" smashed="yes" rot="R90">
 <attribute name="NAME" x="32.766" y="14.097" size="0.8128" layer="25" font="vector" ratio="12" rot="R180"/>
 <attribute name="VALUE" x="34.29" y="10.16" size="1.27" layer="27" rot="R90"/>
@@
 <attribute name="VALUE" x="33.02" y="8.89" size="1.27" layer="27"/>
 </element>
-<element name="R12" library="rcl" package="R0603" value="" x="31.75" y="16.51" smashed="yes" rot="R90">
+<element name="R12" library="rcl" package="R0603" value="1k2" x="31.75" y="16.51" smashed="yes" rot="R90">
 <attribute name="NAME" x="32.766" y="19.177" size="0.8128" layer="25" font="vector" ratio="12" rot="R180"/>
 <attribute name="VALUE" x="34.29" y="15.24" size="1.27" layer="27" rot="R90"/>
@@
 <attribute name="VALUE" x="33.02" y="13.97" size="1.27" layer="27"/>
 </element>
-<element name="R13" library="rcl" package="R0603" value="" x="31.75" y="21.59" smashed="yes" rot="R90">
+<element name="R13" library="rcl" package="R0603" value="1k2" x="31.75" y="21.59" smashed="yes" rot="R90">
 <attribute name="NAME" x="32.766" y="24.257" size="0.8128" layer="25" font="vector" ratio="12" rot="R180"/>
 <attribute name="VALUE" x="34.29" y="20.32" size="1.27" layer="27" rot="R90"/>
