File: V1/usb tester.sch (EAGLE design)
At the start: 34 parts, among them T1 BC847, T2 BC847, T3 BC847, T4 BC847

Commit message: values
Parts:
- R1, R10, R11, R12, R13, R2, R3, R4: value (none) -> 1k2
- R5, R6, R7, R8, R9: value (none) -> 4k7
Changed lines of the file:
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@@
 </classes>
 <parts>
-<part name="R1" library="rcl" deviceset="R-EU_" device="R0603"/>
-<part name="R2" library="rcl" deviceset="R-EU_" device="R0603"/>
-<part name="R3" library="rcl" deviceset="R-EU_" device="R0603"/>
-<part name="R4" library="rcl" deviceset="R-EU_" device="R0603"/>
+<part name="R1" library="rcl" deviceset="R-EU_" device="R0603" value="1k2"/>
+<part name="R2" library="rcl" deviceset="R-EU_" device="R0603" value="1k2"/>
+<part name="R3" library="rcl" deviceset="R-EU_" device="R0603" value="1k2"/>
+<part name="R4" library="rcl" deviceset="R-EU_" device="R0603" value="1k2"/>
 <part name="JP1" library="SparkFun-Connectors" deviceset="USB" device="-A-SMD"/>
 <part name="T1" library="transistor" deviceset="BC847" device=""/>
@@
 <part name="T3" library="transistor" deviceset="BC847" device=""/>
 <part name="T4" library="transistor" deviceset="BC847" device=""/>
-<part name="R5" library="rcl" deviceset="R-EU_" device="R0603"/>
-<part name="R6" library="rcl" deviceset="R-EU_" device="R0603"/>
-<part name="R7" library="rcl" deviceset="R-EU_" device="R0603"/>
-<part name="R8" library="rcl" deviceset="R-EU_" device="R0603"/>
+<part name="R5" library="rcl" deviceset="R-EU_" device="R0603" value="4k7"/>
+<part name="R6" library="rcl" deviceset="R-EU_" device="R0603" value="4k7"/>
+<part name="R7" library="rcl" deviceset="R-EU_" device="R0603" value="4k7"/>
+<part name="R8" library="rcl" deviceset="R-EU_" device="R0603" value="4k7"/>
 <part name="P+1" library="supply1" deviceset="VCC" device=""/>
 <part name="L1" library="led" deviceset="LED" device="CHIPLED_0805"/>
@@
 <part name="L4" library="led" deviceset="LED" device="CHIPLED_0805"/>
 <part name="AVRISP" library="SparkFun-Connectors" deviceset="AVR_SPI_PRG_6" device="2X3_LOCK"/>
-<part name="R9" library="rcl" deviceset="R-EU_" device="R0603"/>
+<part name="R9" library="rcl" deviceset="R-EU_" device="R0603" value="4k7"/>
 <part name="GND4" library="supply1" deviceset="GND" device=""/>
 <part name="JP3" library="SparkFun-Connectors" deviceset="USB" device="-A-SMD"/>
-<part name="R10" library="rcl" deviceset="R-EU_" device="R0603"/>
+<part name="R10" library="rcl" deviceset="R-EU_" device="R0603" value="1k2"/>
 <part name="L5" library="led" deviceset="LED" device="CHIPLED_0805"/>
-<part name="R11" library="rcl" deviceset="R-EU_" device="R0603"/>
+<part name="R11" library="rcl" deviceset="R-EU_" device="R0603" value="1k2"/>
 <part name="L6" library="led" deviceset="LED" device="CHIPLED_0805"/>
-<part name="R12" library="rcl" deviceset="R-EU_" device="R0603"/>
+<part name="R12" library="rcl" deviceset="R-EU_" device="R0603" value="1k2"/>
 <part name="L7" library="led" deviceset="LED" device="CHIPLED_0805"/>
-<part name="R13" library="rcl" deviceset="R-EU_" device="R0603"/>
+<part name="R13" library="rcl" deviceset="R-EU_" device="R0603" value="1k2"/>
 <part name="L8" library="led" deviceset="LED" device="CHIPLED_0805"/>
 <part name="P+4" library="supply1" deviceset="VCC" device=""/>
@@
 <pinref part="JP1" gate="G$1" pin="VBUS"/>
 <wire x1="119.38" y1="73.66" x2="119.38" y2="68.58" width="0.1524" layer="91"/>
-<wire x1="119.38" y1="68.58" x2="119.38" y2="53.34" width="0.1524" layer="91"/>
 <wire x1="119.38" y1="68.58" x2="106.68" y2="68.58" width="0.1524" layer="91"/>
 <junction x="119.38" y="68.58"/>
 <label x="106.68" y="68.58" size="1.016" layer="95" rot="R180" xref="yes"/>
+<pinref part="JP2" gate="G$1" pin="VCC"/>
+<wire x1="119.38" y1="22.86" x2="119.38" y2="68.58" width="0.1524" layer="91"/>
 </segment>
 <segment>
@@
 <wire x1="76.2" y1="78.74" x2="76.2" y2="63.5" width="0.1524" layer="91"/>
 </segment>
-<segment>
-<pinref part="JP2" gate="G$1" pin="VCC"/>
-<wire x1="119.38" y1="22.86" x2="119.38" y2="53.34" width="0.1524" layer="91"/>
-</segment>
 </net>
 <net name="CABLE_DMINUS" class="0">
@@
 <pinref part="JP1" gate="G$1" pin="D-"/>
 <wire x1="116.84" y1="73.66" x2="116.84" y2="66.04" width="0.1524" layer="91"/>
-<wire x1="116.84" y1="66.04" x2="116.84" y2="53.34" width="0.1524" layer="91"/>
 <wire x1="116.84" y1="66.04" x2="106.68" y2="66.04" width="0.1524" layer="91"/>
 <junction x="116.84" y="66.04"/>
 <label x="106.68" y="66.04" size="1.016" layer="95" rot="R180" xref="yes"/>
+<pinref part="JP2" gate="G$1" pin="D-"/>
+<wire x1="116.84" y1="22.86" x2="116.84" y2="66.04" width="0.1524" layer="91"/>
 </segment>
 <segment>
@@
 <wire x1="76.2" y1="38.1" x2="76.2" y2="22.86" width="0.1524" layer="91"/>
 </segment>
-<segment>
-<pinref part="JP2" gate="G$1" pin="D-"/>
-<wire x1="116.84" y1="22.86" x2="116.84" y2="53.34" width="0.1524" layer="91"/>
-</segment>
 </net>
 <net name="CABLE_DPLUS" class="0">
@@
 <pinref part="JP1" gate="G$1" pin="D+"/>
 <wire x1="114.3" y1="73.66" x2="114.3" y2="63.5" width="0.1524" layer="91"/>
-<wire x1="114.3" y1="63.5" x2="114.3" y2="53.34" width="0.1524" layer="91"/>
 <wire x1="114.3" y1="63.5" x2="106.68" y2="63.5" width="0.1524" layer="91"/>
 <junction x="114.3" y="63.5"/>
 <label x="106.68" y="63.5" size="1.016" layer="95" rot="R180" xref="yes"/>
+<pinref part="JP2" gate="G$1" pin="D+"/>
+<wire x1="114.3" y1="22.86" x2="114.3" y2="63.5" width="0.1524" layer="91"/>
 </segment>
 <segment>
@@
 <pinref part="T4" gate="G$1" pin="C"/>
 <wire x1="35.56" y1="22.86" x2="35.56" y2="38.1" width="0.1524" layer="91"/>
-</segment>
-<segment>
-<pinref part="JP2" gate="G$1" pin="D+"/>
-<wire x1="114.3" y1="22.86" x2="114.3" y2="53.34" width="0.1524" layer="91"/>
 </segment>
 </net>
@@
 </sheet>
 </sheets>
+<errors>
+</errors>
 </schematic>
 </drawing>
